File: $analog-board.sch (KiCad schematic (older format))
At the start: 502 parts, among them J1 AC IN, J2 OUT, J3 CONN_20X2, P2 CONN_01X02, Q1 2N3906, Q10 2N3906, Q11 2N3906, Q12 2N3906, Q13 2N3906, Q14 2N3906, Q15 2N3906, Q16 2N3906, Q17 NPN, Q18 NPN, Q19 J111, Q2 2N3906, Q20 2N3906, Q3 2N3906, Q4 2N3906, Q5 2N3906, Q6 BCM857BS, Q7 2N3906, Q8 2N3906, Q9 2N3906, U1 LM13700, U10 ADR01, U11 DG212B, U12 DG212B, U13 DG408, U14 DG408, U15 TL072-, U16 DG408, U17 DG408, U18 LM13700, U19 LM13700, U2 LM13700, U20 74HC75, U21 TL072-, U22 TL074-, U23 TL074-, U24 TL074-, U25 TL074-, U26 TL072-, U27 TL074-, U28 TL074-, U29 LM13700, U3 LM13700, U30 LM13700, U31 TL074-, U32 LM13700, U33 TL074-, U34 TL074-, U35 TL074-, U36 74LV573, U38 0 - 10V, U39 TL074-, U4 DG212B, U40 DG419, U41 0 - 10V, U42 10 - 0V, U43 LM7812, U44 LM7912, U45 DG408, U46 7805, U5 TL074-, U6 AD5556, U7 TL072-, U8 TL074-, U9 AD8672

Commit message: just added a few notes about removing filter pitch depth control VCA and maybe repurposing OTA for Mike Simms dual OTA VCA for final volume VCA
Other:
- note added: "PITCH MODULATION OF FILTER IS NOW IRRELEVANT:\nIt is now integrated with filter cutoff CV. This whole section\ncan be deleted and components used for other features. \nPerhaps a Mike Simms dual OTA VCA for final volume VCA?"
- note removed: "PITCH MODULATION OF FILTER IS NOW IRRELEVANT:\nIt is now integrated with filter cutoff CV. This whole section\ncan be deleted and components used for other features. \nPerhaps a Scott Sites dual OTA VCA for final volume VCA?"
Changed lines of the file:
@@
 	22850 7600 22850 4400
 Text Notes 22900 4800 0    60   ~ 0
-PITCH MODULATION OF FILTER IS NOW IRRELEVANT:\nIt is now integrated with filter cutoff CV. This whole section\ncan be deleted and components used for other features. \nPerhaps a Scott Sites dual OTA VCA for final volume VCA?
+PITCH MODULATION OF FILTER IS NOW IRRELEVANT:\nIt is now integrated with filter cutoff CV. This whole section\ncan be deleted and components used for other features. \nPerhaps a Mike Simms dual OTA VCA for final volume VCA?
 Text Notes 32950 14050 0    60   ~ 0
 THIS VCF SCALE TRIMMER MAY\nNOT BE REQUIRED NOW THAT\nFILTER TRACKING IS AUTOTUNED?
